File: Schematics/Sensore Corrente.sch (KiCad schematic (older format))
At the start: 17 parts, among them P1 Programmazione (5 PIN), P2 Antenna (2 PIN), P3 Sensore corrente (2 PIN), SW1 SW_PUSH, SW2 DIP, U1 PIC16F1518, U2 TRX_32000985

Commit message: 29-09-2017
Parts:
- removed D3: 3.3, ~, symbol ZENER
- added D3: SR102, ~, symbol DIODESCH
- added R4: 10k, ~, symbol R
- added R6, R7: 33.2, ~, symbol R
- added U3: MCP6N16, ~, symbol MCP6N16
- renumbered R4 to R3, R3 to R5
Connections:
- net GND: now also R4.2, U3.4 (Vss); no longer D4.1 (A), P3.1 (P1), R5.2
- net VDD: now also D4.2 (K), D3.2 (K), U3.8 (Vdd)
- net at U1.11 (RC0/T1OSO/T1CKI): now also R4.1, U3.1 (EN)
- new net: U1.4 (RA2/AN2/VREF-/CVREF/C2IN+), U3.6 (Vfg), U3.7 (Vout)
- new net: R5.1, R6.2
- new net: D4.1 (A), P3.1 (P1), R5.2, U3.2 (Vim(-))
- new net: D3.1 (A), P3.2 (PM), R7.1, U3.3 (Vip(+))
- new net: R6.1, R7.2
Other:
- note added: "Gdm=1 -> Rf=0, Rg=open"
- moved on the sheet: BT1, D1, D2, D4, DL1, P1, P2, P3, R1, R2, R3, R5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
